Commit message: Made the rpy of one joint different to now be on the other side

File: R_inspire_fullpath2.urdf (robot description, URDF)
Before this commit: robot R_inspire, 11 links, 10 joints
Joints:
- joint R_index_proximal_yaw_joint: origin xyz=-0.01696 -0.0691 0.02045 rpy=1.5708 -1.5708 0 -> xyz=-0.01696 -0.0691 0.02045 rpy=1.0 0.0 0.0

Commit message: pitch joints now face each other to make a claw

File: R_inspire_fullpath2.urdf (robot description, URDF)
Before this commit: robot R_inspire, 11 links, 10 joints
Joints:
- joint R_index_proximal_pitch_joint: origin xyz=-0.0088099 0.010892 -0.00925 rpy=1.5708 0 2.8587 -> xyz=-0.0088099 0.010892 -0.00925 rpy=0 0 ${-pi}
- joint R_thumb_proximal_pitch_joint: origin xyz=-0.0088099 0.010892 -0.00925 rpy=1.5708 0 2.8587 -> xyz=-0.0088099 0.010892 -0.00925 rpy=0.0 ${pi} 0.0

Commit message: Made the thumbs more parallel to each other

File: R_inspire_fullpath2.urdf (robot description, URDF)
Before this commit: robot R_inspire, 11 links, 10 joints
Joints:
- joint R_index_proximal_yaw_joint: origin xyz=-0.01696 -0.0691 0.02045 rpy=1.0 0.0 0.0 -> xyz=-0.01696 -0.0771 0.02045 rpy=1.39 0.0006 0.024

Commit message: Took out all the pi since Isaac Sim can't parse it to 3.14

File: R_inspire_fullpath2.urdf (robot description, URDF)
Before this commit: robot R_inspire, 11 links, 10 joints
Joints:
- joint R_index_proximal_pitch_joint: origin xyz=-0.0088099 0.010892 -0.00925 rpy=0 0 ${-pi} -> xyz=-0.0088099 0.010892 -0.00925 rpy=0 0 -3.14
- joint R_index_proximal_yaw_joint: axis 0 0 -1 -> 0 0 1
- joint R_thumb_proximal_pitch_joint: origin xyz=-0.0088099 0.010892 -0.00925 rpy=0.0 ${pi} 0.0 -> xyz=-0.0088099 0.010892 -0.00925 rpy=0.0 3.14 0.0
- joint R_thumb_proximal_yaw_joint: axis 0 0 -1 -> 0 0 1
